File: Electrical/KiCad/Light-Up Hat/Light-Up Hat.sch (KiCad schematic (older format))
At the start: 19 parts

Commit message: PCB For Manufacture
Parts:
- removed D?: D_Zener, symbol Device:D_Zener
- removed D? (x2): D_Schottky, symbol Device:D_Schottky
- removed J?: Conn_01x05, symbol Connector_Generic:Conn_01x05
- removed JP?: Jumper_NO_Small, symbol Device:Jumper_NO_Small
- removed Q? (x2): 2N3904, Package_TO_SOT_THT:TO-92_Inline, symbol Transistor_BJT:2N3904
- removed R? (x2): 100KΩ, symbol Device:R_Small
- removed R?: R, symbol Device:R
- removed SW?: SW_Push_Dual, symbol Switch:SW_Push_Dual
- added C1, C2: 1μF, Capacitor_SMD:C_0805_2012Metric, symbol Device:C_Small
- added C3: C_Small, Capacitor_SMD:C_0805_2012Metric, symbol Device:C_Small
- added J1: Conn_01x04, Connector_PinHeader_2.54mm:PinHeader_1x04_P2.54mm_Vertical, symbol Connector_Generic:Conn_01x04
- added Q1: 2N3906, Package_TO_SOT_SMD:SOT-23, symbol Transistor_BJT:2N3906
- added SW1: SW_SPST, Button_Switch_THT:SW_PUSH_8mm_H5mm, symbol Switch:SW_SPST
- added U1: AP1117-33, Package_TO_SOT_SMD:SOT-23, symbol Regulator_Linear:AP1117-33
- BT1: renamed from BT?; footprint (none) -> Connector_Wire:SolderWirePad_1x02_P5.08mm_Drill1.5mm
- D1, D2, D3, D4, D5: renamed from D?; footprint (none) -> LED_THT:LED_D5.0mm
- R1: renamed from R?; value R_Small -> 1KΩ; footprint (none) -> Resistor_SMD:R_0805_2012Metric
- gave numbers to parts that had none: 1
Connections:
- net labels removed: ADC, VDD
- wire segments 27 -> 18
Other:
- note removed: "POWER SUPPLY"

Commit message: Hat LEDs blink on and off every 1 second
Parts:
- removed Q1: 2N3906, Package_TO_SOT_SMD:SOT-23, symbol Transistor_BJT:2N3906
- added Q1: MMBT3906, Package_TO_SOT_SMD:SOT-23, symbol Transistor_BJT:MMBT3906
Changed lines of the file:
@@
 	1    0    0    -1
 $EndComp
+Wire Wire Line
+	2700 5100 3050 5100
 $Comp
-L Transistor_BJT:2N3906 Q1
-U 1 1 5DB0F78B
+L Transistor_BJT:MMBT3906 Q1
+U 1 1 5DD09D79
 P 2600 4900
 F 0 "Q1" H 2791 4854 50  0000 L CNN
-F 1 "2N3906" H 2791 4945 50  0000 L CNN
+F 1 "MMBT3906" H 2791 4945 50  0000 L CNN
 F 2 "Package_TO_SOT_SMD:SOT-23" H 2800 4825 50  0001 L CIN
 F 3 "https://www.fairchildsemi.com/datasheets/2N/2N3906.pdf" H 2600 4900 50  0001 L CNN
@@
 	1    0    0    1
 $EndComp
-Wire Wire Line
-	2700 5100 3050 5100
 $EndSCHEMATC

Commit message: fixed board design for new revision
Parts:
- removed U2: PIC10F220-IOT, Package_TO_SOT_SMD:SOT-23-6, symbol MCU_Microchip_PIC10:PIC10F220-IOT
- added U2: PIC10F200-IOT, Package_TO_SOT_SMD:SOT-23-6, symbol MCU_Microchip_PIC10:PIC10F200-IOT
- C1, C2: LCSC (none) -> C28323
- C3: LCSC (none) -> C49678
- Q1: LCSC (none) -> C2143
- R1: LCSC (none) -> C17513
- U1: value AP1117-33 -> XC6206; LCSC (none) -> C5446
Changed lines of the file:
@@
 $EndDescr
-$Comp
-L MCU_Microchip_PIC10:PIC10F220-IOT U2
-U 1 1 5DAB79AC
-P 6300 3400
-F 0 "U2" H 6650 4000 50  0000 C CNN
-F 1 "PIC10F220-IOT" H 6650 3900 50  0000 C CNN
-F 2 "Package_TO_SOT_SMD:SOT-23-6" H 6350 4050 50  0001 L CIN
-F 3 "http://ww1.microchip.com/downloads/en/DeviceDoc/41270E.pdf" H 6300 3400 50  0001 C CNN
-	1    6300 3400
-	1    0    0    -1
-$EndComp
 $Comp
 L power:GND #PWR09
@@
 F 2 "Resistor_SMD:R_0805_2012Metric" H 2300 4900 50  0001 C CNN
 F 3 "~" H 2300 4900 50  0001 C CNN
+F 4 "C17513" V 2300 4900 50  0001 C CNN "LCSC"
 	1    2300 4900
 	0    1    -1   0
@@
 P 2350 1250
 F 0 "U1" H 2350 1492 50  0000 C CNN
-F 1 "AP1117-33" H 2350 1401 50  0000 C CNN
+F 1 "XC6206" H 2350 1401 50  0000 C CNN
 F 2 "Package_TO_SOT_SMD:SOT-23" H 2350 1450 50  0001 C CNN
 F 3 "http://www.diodes.com/datasheets/AP1117.pdf" H 2450 1000 50  0001 C CNN
+F 4 "C5446" H 2350 1250 50  0001 C CNN "LCSC"
 	1    2350 1250
 	1    0    0    -1
@@
 F 2 "Capacitor_SMD:C_0805_2012Metric" H 1900 1400 50  0001 C CNN
 F 3 "~" H 1900 1400 50  0001 C CNN
+F 4 "C28323" H 1900 1400 50  0001 C CNN "LCSC"
 	1    1900 1400
 	1    0    0    -1
@@
 F 2 "Capacitor_SMD:C_0805_2012Metric" H 2800 1400 50  0001 C CNN
 F 3 "~" H 2800 1400 50  0001 C CNN
+F 4 "C28323" H 2800 1400 50  0001 C CNN "LCSC"
 	1    2800 1400
 	1    0    0    -1
@@
 F 2 "Capacitor_SMD:C_0805_2012Metric" H 6850 3900 50  0001 C CNN
 F 3 "~" H 6850 3900 50  0001 C CNN
+F 4 "C49678" H 6850 3900 50  0001 C CNN "LCSC"
 	1    6850 3900
 	1    0    0    -1
@@
 Wire Wire Line
 	6300 4000 6850 4000
-Connection ~ 6300 4000
 $Comp
 L power:+3.3V #PWR010
@@
 F 2 "Package_TO_SOT_SMD:SOT-23" H 2800 4825 50  0001 L CIN
 F 3 "https://www.fairchildsemi.com/datasheets/2N/2N3906.pdf" H 2600 4900 50  0001 L CNN
+F 4 "C2143" H 2600 4900 50  0001 C CNN "LCSC"
 	1    2600 4900
 	1    0    0    1
 $EndComp
+$Comp
+L MCU_Microchip_PIC10:PIC10F200-IOT U2
+U 1 1 5DD30468
+P 6300 3400
+F 0 "U2" H 6300 4178 50  0000 C CNN
+F 1 "PIC10F200-IOT" H 6300 4087 50  0000 C CNN
+F 2 "Package_TO_SOT_SMD:SOT-23-6" H 6350 4050 50  0001 L CIN
+F 3 "http://ww1.microchip.com/downloads/en/DeviceDoc/41239D.pdf" H 6300 3400 50  0001 C CNN
+F 4 "C8224" H 6300 3400 50  0001 C CNN "LCSC"
+	1    6300 3400
+	1    0    0    -1
+$EndComp
+Connection ~ 6300 4000
 $EndSCHEMATC
